File: 66_ekip.kicad_pcb (KiCad board)
At the start: 0 parts

Commit message: Matrix routed on the PCB
Parts:
- added C1: 22p, Capacitor_SMD:C_0805_2012Metric, B.Cu at (-201.9, 127.4)
- added C10: 0.1u, Capacitor_SMD:C_0805_2012Metric, B.Cu at (-178.2, 152.8)
- added C11: 0.1u, Capacitor_SMD:C_0805_2012Metric, B.Cu at (-180.3, 146.8)
- added C12: 10u, Capacitor_SMD:C_0805_2012Metric, B.Cu at (-184.8, 143.8)
- added C13: 10u, Capacitor_SMD:C_0805_2012Metric, B.Cu at (-184.8, 140.8)
- added C14: 100nF, Capacitor_SMD:C_0805_2012Metric, B.Cu at (-180.3, 143.8)
- added C2: 22p, Capacitor_SMD:C_0805_2012Metric, B.Cu at (-189.2, 138.7)
- added C3: 1u, Capacitor_SMD:C_0805_2012Metric, B.Cu at (-189.2, 141.7)
- added C4: 10u, Capacitor_SMD:C_0805_2012Metric, B.Cu at (-197.4, 127.4)
- added C5: 1u, Capacitor_SMD:C_0805_2012Metric, B.Cu at (-201.9, 130.4)
- added C6: 10u, Capacitor_SMD:C_0805_2012Metric, B.Cu at (-163.4, 155.1)
- added C7: 1u, Capacitor_SMD:C_0805_2012Metric, B.Cu at (-180.3, 140.8)
- added C8: 0.1u, Capacitor_SMD:C_0805_2012Metric, B.Cu at (-193.2, 134.0)
- added C9: 0.1u, Capacitor_SMD:C_0805_2012Metric, B.Cu at (-178.2, 149.8)
- added D1: D_Small, Diode_SMD:D_0805_2012Metric, B.Cu at (-7.94, 68.3)
- added D10: D_Small, Diode_SMD:D_0805_2012Metric, B.Cu at (163.5, 68.3)
- added D11: D_Small, Diode_SMD:D_0805_2012Metric, B.Cu at (182.6, 68.3)
- added D12: D_Small, Diode_SMD:D_0805_2012Metric, B.Cu at (201.6, 68.4)
- added D13: D_Small, Diode_SMD:D_0805_2012Metric, B.Cu at (220.7, 68.4)
- added D14: D_Small, Diode_SMD:D_0805_2012Metric, B.Cu at (239.7, 68.3)
- added D15: D_Small, Diode_SMD:D_0805_2012Metric, B.Cu at (249.2, 68.4)
- added D16: D_Small, Diode_SMD:D_0805_2012Metric, B.Cu at (287.3, 68.1)
- added D17: D_Small, Diode_SMD:D_0805_2012Metric, B.Cu at (-3.17, 87.5)
- added D18: D_Small, Diode_SMD:D_0805_2012Metric, B.Cu at (20.6, 87.3)
- added D19: D_Small, Diode_SMD:D_0805_2012Metric, B.Cu at (39.7, 87.3)
- added D2: D_Small, Diode_SMD:D_0805_2012Metric, B.Cu at (11.1, 68.3)
- added D20: D_Small, Diode_SMD:D_0805_2012Metric, B.Cu at (58.7, 87.3)
- added D21: D_Small, Diode_SMD:D_0805_2012Metric, B.Cu at (77.8, 87.3)
- added D22: D_Small, Diode_SMD:D_0805_2012Metric, B.Cu at (96.8, 87.3)
- added D23: D_Small, Diode_SMD:D_0805_2012Metric, B.Cu at (115.9, 87.3)
- added D24: D_Small, Diode_SMD:D_0805_2012Metric, B.Cu at (134.9, 87.5)
- added D25: D_Small, Diode_SMD:D_0805_2012Metric, B.Cu at (154.0, 87.5)
- added D26: D_Small, Diode_SMD:D_0805_2012Metric, B.Cu at (173.0, 87.3)
- added D27: D_Small, Diode_SMD:D_0805_2012Metric, B.Cu at (192.1, 87.5)
- added D28: D_Small, Diode_SMD:D_0805_2012Metric, B.Cu at (211.1, 87.5)
- added D29: D_Small, Diode_SMD:D_0805_2012Metric, B.Cu at (230.2, 87.3)
- added D3: D_Small, Diode_SMD:D_0805_2012Metric, B.Cu at (30.2, 68.3)
- added D30: D_Small, Diode_SMD:D_0805_2012Metric, B.Cu at (254.0, 87.5)
- added D31: D_Small, Diode_SMD:D_0805_2012Metric, B.Cu at (287.3, 87.5)
- added D32: D_Small, Diode_SMD:D_0805_2012Metric, B.Cu at (5.56, 106.5)
- added D33: D_Small, Diode_SMD:D_0805_2012Metric, B.Cu at (25.4, 106.4)
- added D34: D_Small, Diode_SMD:D_0805_2012Metric, B.Cu at (44.5, 106.5)
- added D35: D_Small, Diode_SMD:D_0805_2012Metric, B.Cu at (63.5, 106.5)
- added D36: D_Small, Diode_SMD:D_0805_2012Metric, B.Cu at (82.5, 106.4)
- added D37: D_Small, Diode_SMD:D_0805_2012Metric, B.Cu at (101.6, 106.4)
- added D38: D_Small, Diode_SMD:D_0805_2012Metric, B.Cu at (120.7, 106.5)
- added D39: D_Small, Diode_SMD:D_0805_2012Metric, B.Cu at (139.7, 106.4)
- added D4: D_Small, Diode_SMD:D_0805_2012Metric, B.Cu at (49.2, 68.3)
- added D40: D_Small, Diode_SMD:D_0805_2012Metric, B.Cu at (158.8, 106.4)
- added D41: D_Small, Diode_SMD:D_0805_2012Metric, B.Cu at (177.8, 106.5)
- added D42: D_Small, Diode_SMD:D_0805_2012Metric, B.Cu at (196.8, 106.5)
- added D43: D_Small, Diode_SMD:D_0805_2012Metric, B.Cu at (215.9, 106.4)
- added D44: D_Small, Diode_SMD:D_0805_2012Metric, B.Cu at (234.9, 106.4)
- added D45: D_Small, Diode_SMD:D_0805_2012Metric, B.Cu at (246.9, 106.4)
- added D46: D_Small, Diode_SMD:D_0805_2012Metric, B.Cu at (287.3, 106.5)
- added D47: D_Small, Diode_SMD:D_0805_2012Metric, B.Cu at (3.97, 125.4)
- added D48: D_Small, Diode_SMD:D_0805_2012Metric, B.Cu at (15.9, 125.6)
- added D49: D_Small, Diode_SMD:D_0805_2012Metric, B.Cu at (34.9, 125.4)
- added D5: D_Small, Diode_SMD:D_0805_2012Metric, B.Cu at (68.3, 68.3)
- added D50: D_Small, Diode_SMD:D_0805_2012Metric, B.Cu at (54.0, 125.6)
- added D51: D_Small, Diode_SMD:D_0805_2012Metric, B.Cu at (73.0, 125.4)
- added D52: D_Small, Diode_SMD:D_0805_2012Metric, B.Cu at (92.1, 125.4)
- added D53: D_Small, Diode_SMD:D_0805_2012Metric, B.Cu at (111.1, 125.6)
- added D54: D_Small, Diode_SMD:D_0805_2012Metric, B.Cu at (130.2, 125.6)
- added D55: D_Small, Diode_SMD:D_0805_2012Metric, B.Cu at (149.2, 125.4)
- added D56: D_Small, Diode_SMD:D_0805_2012Metric, B.Cu at (168.3, 125.4)
- added D57: D_Small, Diode_SMD:D_0805_2012Metric, B.Cu at (187.3, 125.6)
- added D58: D_Small, Diode_SMD:D_0805_2012Metric, B.Cu at (206.4, 125.4)
- added D59: D_Small, Diode_SMD:D_0805_2012Metric, B.Cu at (232.6, 125.6)
- added D6: D_Small, Diode_SMD:D_0805_2012Metric, B.Cu at (87.3, 68.4)
- added D60: D_Small, Diode_SMD:D_0805_2012Metric, B.Cu at (287.3, 125.4)
- added D61: D_Small, Diode_SMD:D_0805_2012Metric, B.Cu at (263.5, 130.2)
- added D62: D_Small, Diode_SMD:D_0805_2012Metric, B.Cu at (34.9, 144.5)
- added D63: D_Small, Diode_SMD:D_0805_2012Metric, B.Cu at (56.4, 144.6)
- added D64: D_Small, Diode_SMD:D_0805_2012Metric, B.Cu at (127.8, 144.5)
- added D65: D_Small, Diode_SMD:D_0805_2012Metric, B.Cu at (196.8, 144.5)
- added D66: D_Small, Diode_SMD:D_0805_2012Metric, B.Cu at (218.3, 144.6)
- added D67: D_Small, Diode_SMD:D_0805_2012Metric, B.Cu at (244.5, 149.2)
- added D68: D_Small, Diode_SMD:D_0805_2012Metric, B.Cu at (263.5, 149.2)
- added D69: D_Small, Diode_SMD:D_0805_2012Metric, B.Cu at (282.6, 149.4)
- added D7: D_Small, Diode_SMD:D_0805_2012Metric, B.Cu at (106.4, 68.3)
- added D70: D_Small, Diode_SMD:D_0805_2012Metric, B.Cu at (-184.8, 146.8)
- added D71: LED, LED_SMD:LED_0805_2012Metric, B.Cu at (-197.5, 130.4)
- added D72: WS2812, LED_SMD:LED_WS2812_PLCC6_5.0x5.0mm_P1.6mm, B.Cu at (-191.0, 129.2)
- added D73: WS2812, LED_SMD:LED_WS2812_PLCC6_5.0x5.0mm_P1.6mm, B.Cu at (-182.6, 129.2)
- added D74: WS2812, LED_SMD:LED_WS2812_PLCC6_5.0x5.0mm_P1.6mm, B.Cu at (-165.5, 143.7)
- added D75: WS2812, LED_SMD:LED_WS2812_PLCC6_5.0x5.0mm_P1.6mm, B.Cu at (-181.9, 136.0)
- added D76: WS2812, LED_SMD:LED_WS2812_PLCC6_5.0x5.0mm_P1.6mm, B.Cu at (-165.5, 150.3)
- added D77: WS2812, LED_SMD:LED_WS2812_PLCC6_5.0x5.0mm_P1.6mm, B.Cu at (-173.9, 143.6)
- added D78: D_Small, Diode_SMD:D_0805_2012Metric, B.Cu at (89.7, 144.5)
- added D79: D_Small, Diode_SMD:D_0805_2012Metric, B.Cu at (175.4, 144.5)
- added D8: D_Small, Diode_SMD:D_0805_2012Metric, B.Cu at (125.4, 68.4)
- added D9: D_Small, Diode_SMD:D_0805_2012Metric, B.Cu at (144.5, 68.4)
- added J1: BT LE, Connector_PinHeader_1.00mm:PinHeader_1x09_P1.00mm_Vertical, B.Cu at (-167.2, 127.4)
- added J2: AVR-ISP-6, Random_Keyb_Parts:Reset_Pretty, B.Cu at (-172.8, 150.8)
- added J3: JST, Connector_JST:JST_SH_SM04B-SRSS-TB_1x04-1MP_P1.00mm_Horizontal, B.Cu at (-173.3, 136.5)
- added J4: BAT JST, Connector_JST:JST_PH_S2B-PH-SM4-TB_1x02-1MP_P2.00mm_Horizontal, B.Cu at (-156.2, 146.0)
- added R1: 22, Resistor_SMD:R_0805_2012Metric, B.Cu at (-189.2, 144.7)
- added R2: 22, Resistor_SMD:R_0805_2012Metric, B.Cu at (-193.7, 140.0)
- added R3: 100k, Resistor_SMD:R_0805_2012Metric, B.Cu at (-197.6, 133.4)
- added R4: 10k, Resistor_SMD:R_0805_2012Metric, B.Cu at (-182.6, 152.8)
- added R5: 1k, Resistor_SMD:R_0805_2012Metric, B.Cu at (-198.1, 136.4)
- added R6: 10k, Resistor_SMD:R_0805_2012Metric, B.Cu at (-193.7, 137.0)
- added R7: 10k, Resistor_SMD:R_0805_2012Metric, B.Cu at (-178.2, 155.8)
- added R8: 480, Resistor_SMD:R_0805_2012Metric, B.Cu at (-182.6, 149.8)
- added SW1: Esc, MX_Alps_Hybrid:MX-1U-NoLED, F.Cu at (-4.76, 65.1)
- added SW10: 9, MX_Alps_Hybrid:MX-1U-NoLED, F.Cu at (166.7, 65.1)
- added SW11: 0, MX_Alps_Hybrid:MX-1U-NoLED, F.Cu at (185.7, 65.1)
- added SW12: -, MX_Alps_Hybrid:MX-1U-NoLED, F.Cu at (204.8, 65.1)
- added SW13: =, MX_Alps_Hybrid:MX-1U-NoLED, F.Cu at (223.8, 65.1)
- added SW14: \ 1u, MX_Alps_Hybrid:MX-1U-NoLED, F.Cu at (242.9, 65.1)
- added SW15: Backspace, MX_Alps_Hybrid:MX-2U-NoLED, F.Cu at (252.4, 65.1)
- added SW16: Col R1, MX_Alps_Hybrid:MX-1U-NoLED, F.Cu at (290.5, 65.1)
- added SW17: Backtick 1u, MX_Alps_Hybrid:MX-1U-NoLED, F.Cu at (261.9, 65.1)
- added SW18: Tab, MX_Alps_Hybrid:MX-1.5U-NoLED, F.Cu at (0.00, 84.1)
- added SW19: Q, MX_Alps_Hybrid:MX-1U-NoLED, F.Cu at (23.8, 84.1)
- added SW2: 1, MX_Alps_Hybrid:MX-1U-NoLED, F.Cu at (14.3, 65.1)
- added SW20: W, MX_Alps_Hybrid:MX-1U-NoLED, F.Cu at (42.9, 84.1)
- added SW21: E, MX_Alps_Hybrid:MX-1U-NoLED, F.Cu at (61.9, 84.1)
- added SW22: R, MX_Alps_Hybrid:MX-1U-NoLED, F.Cu at (81.0, 84.1)
- added SW23: T, MX_Alps_Hybrid:MX-1U-NoLED, F.Cu at (100.0, 84.1)
- added SW24: Y, MX_Alps_Hybrid:MX-1U-NoLED, F.Cu at (119.1, 84.1)
- added SW25: U, MX_Alps_Hybrid:MX-1U-NoLED, F.Cu at (138.1, 84.1)
- added SW26: I, MX_Alps_Hybrid:MX-1U-NoLED, F.Cu at (157.2, 84.1)
- added SW27: O, MX_Alps_Hybrid:MX-1U-NoLED, F.Cu at (176.2, 84.1)
- added SW28: P, MX_Alps_Hybrid:MX-1U-NoLED, F.Cu at (195.3, 84.1)
- added SW29: [, MX_Alps_Hybrid:MX-1U-NoLED, F.Cu at (214.3, 84.1)
- added SW3: 2, MX_Alps_Hybrid:MX-1U-NoLED, F.Cu at (33.3, 65.1)
- added SW30: ], MX_Alps_Hybrid:MX-1U-NoLED, F.Cu at (233.4, 84.1)
- added SW31: \ 1.5u, MX_Alps_Hybrid:MX-1.5U-NoLED, F.Cu at (257.2, 84.1)
- added SW32: Col R2, MX_Alps_Hybrid:MX-1U-NoLED, F.Cu at (290.5, 84.1)
- added SW33: Enter ISO, MX_Alps_Hybrid:MX-ISO-ReversedStabilizers-NoLED, F.Cu at (259.6, 93.7)
- added SW34: CapsLock, MX_Alps_Hybrid:MX-1.75U-NoLED, F.Cu at (2.38, 103.2)
- added SW35: A, MX_Alps_Hybrid:MX-1U-NoLED, F.Cu at (28.6, 103.2)
- added SW36: S, MX_Alps_Hybrid:MX-1U-NoLED, F.Cu at (47.6, 103.2)
- added SW37: D, MX_Alps_Hybrid:MX-1U-NoLED, F.Cu at (66.7, 103.2)
- added SW38: F, MX_Alps_Hybrid:MX-1U-NoLED, F.Cu at (85.7, 103.2)
- added SW39: G, MX_Alps_Hybrid:MX-1U-NoLED, F.Cu at (104.8, 103.2)
- added SW4: 3, MX_Alps_Hybrid:MX-1U-NoLED, F.Cu at (52.4, 65.1)
- added SW40: H, MX_Alps_Hybrid:MX-1U-NoLED, F.Cu at (123.8, 103.2)
- added SW41: J, MX_Alps_Hybrid:MX-1U-NoLED, F.Cu at (142.9, 103.2)
- added SW42: K, MX_Alps_Hybrid:MX-1U-NoLED, F.Cu at (161.9, 103.2)
- added SW43: L, MX_Alps_Hybrid:MX-1U-NoLED, F.Cu at (181.0, 103.2)
- added SW44: ;, MX_Alps_Hybrid:MX-1U-NoLED, F.Cu at (200.0, 103.2)
- added SW45: ', MX_Alps_Hybrid:MX-1U-NoLED, F.Cu at (219.1, 103.2)
- added SW46: \ ISO, MX_Alps_Hybrid:MX-1U-NoLED, F.Cu at (238.1, 103.2)
- added SW47: Enter, MX_Alps_Hybrid:MX-2.25U-ReversedStabilizers-NoLED, F.Cu at (250.0, 103.2)
- added SW48: Col R3, MX_Alps_Hybrid:MX-1U-NoLED, F.Cu at (290.5, 103.2)
- added SW49: Shift 1.25 ISO, MX_Alps_Hybrid:MX-1.25U-NoLED, F.Cu at (-2.38, 122.2)
- added SW5: 4, MX_Alps_Hybrid:MX-1U-NoLED, F.Cu at (71.4, 65.1)
- added SW50: Shift 2.25, MX_Alps_Hybrid:MX-2.25U-ReversedStabilizers-NoLED, F.Cu at (7.14, 122.2)
- added SW51: <> ISO, MX_Alps_Hybrid:MX-1U-NoLED, F.Cu at (19.1, 122.2)
- added SW52: Z, MX_Alps_Hybrid:MX-1U-NoLED, F.Cu at (38.1, 122.2)
- added SW53: X, MX_Alps_Hybrid:MX-1U-NoLED, F.Cu at (57.1, 122.2)
- added SW54: C, MX_Alps_Hybrid:MX-1U-NoLED, F.Cu at (76.2, 122.2)
- added SW55: V, MX_Alps_Hybrid:MX-1U-NoLED, F.Cu at (95.2, 122.2)
- added SW56: B, MX_Alps_Hybrid:MX-1U-NoLED, F.Cu at (114.3, 122.2)
- added SW57: N, MX_Alps_Hybrid:MX-1U-NoLED, F.Cu at (133.3, 122.2)
- added SW58: M, MX_Alps_Hybrid:MX-1U-NoLED, F.Cu at (152.4, 122.2)
- added SW59: <, MX_Alps_Hybrid:MX-1U-NoLED, F.Cu at (171.4, 122.2)
- added SW6: 5, MX_Alps_Hybrid:MX-1U-NoLED, F.Cu at (90.5, 65.1)
- added SW60: >, MX_Alps_Hybrid:MX-1U-NoLED, F.Cu at (190.5, 122.2)
- added SW61: /, MX_Alps_Hybrid:MX-1U-NoLED, F.Cu at (209.6, 122.2)
- added SW62: Shift 1.75, MX_Alps_Hybrid:MX-1.75U-NoLED, F.Cu at (235.7, 122.2)
- added SW63: Col R4, MX_Alps_Hybrid:MX-1U-NoLED, F.Cu at (290.5, 122.2)
- added SW64: Up arrow, MX_Alps_Hybrid:MX-1U-NoLED, F.Cu at (266.7, 127.0)
- added SW65: L Super 1.25u, MX_Alps_Hybrid:MX-1.25U-NoLED, F.Cu at (40.5, 141.3)
- added SW66: L Alt 1u, MX_Alps_Hybrid:MX-1U-NoLED, F.Cu at (61.9, 141.3)
- added SW67: R Alt 1u, MX_Alps_Hybrid:MX-1U-NoLED, F.Cu at (200.0, 141.3)
- added SW68: R Super 1.25u, MX_Alps_Hybrid:MX-1.25U-NoLED, F.Cu at (221.5, 141.3)
- added SW69: L Super 1u, MX_Alps_Hybrid:MX-1U-NoLED, F.Cu at (38.1, 141.3)
- added SW7: 6, MX_Alps_Hybrid:MX-1U-NoLED, F.Cu at (109.5, 65.1)
- added SW70: L Alt 1.25u, MX_Alps_Hybrid:MX-1.25U-NoLED, F.Cu at (59.5, 141.3)
- added SW71: Space 6.25u, MX_Alps_Hybrid:MX-6.25U-ReversedStabilizers-NoLED, F.Cu at (131.0, 141.3)
- added SW72: R Alt 1.25u, MX_Alps_Hybrid:MX-1.25U-NoLED, F.Cu at (202.4, 141.3)
- added SW73: R Super 1u, MX_Alps_Hybrid:MX-1U-NoLED, F.Cu at (223.8, 141.3)
- added SW74: Left arrow, MX_Alps_Hybrid:MX-1U-NoLED, F.Cu at (247.7, 146.1)
- added SW75: Down arrow, MX_Alps_Hybrid:MX-1U-NoLED, F.Cu at (266.7, 146.1)
- added SW76: Right arrow, MX_Alps_Hybrid:MX-1U-NoLED, F.Cu at (285.8, 146.1)
- added SW77: SW_Push, Button_Switch_SMD:SW_SPST_SKQG_WithStem, B.Cu at (-173.6, 129.3)
- added SW78: CapsLock Stepped, MX_Alps_Hybrid:MX-1.25U-NoLED, F.Cu at (-2.38, 103.2)
- added SW79: Split Space R 2.75u, MX_Alps_Hybrid:MX-2.75U-ReversedStabilizers-NoLED, F.Cu at (140.5, 141.3)
- added SW8: 7, MX_Alps_Hybrid:MX-1U-NoLED, F.Cu at (128.6, 65.1)
- added SW80: Split Space L 2.25u, MX_Alps_Hybrid:MX-2.25U-ReversedStabilizers-NoLED, F.Cu at (92.9, 141.3)
- added SW81: Mod R 1.25u, MX_Alps_Hybrid:MX-1.25U-NoLED, F.Cu at (178.6, 141.3)
- added SW9: 8, MX_Alps_Hybrid:MX-1U-NoLED, F.Cu at (147.6, 65.1)
- added U1: AP2112K-3.3, Package_TO_SOT_SMD:SOT-23-5, B.Cu at (-188.5, 134.9)
- added U2: ATmega32U4-AU, Package_QFP:TQFP-44_10x10mm_P0.8mm, B.Cu at (-158.3, 133.1)
- added U3: MCP73831-2-OT, Package_TO_SOT_SMD:SOT-23-5, B.Cu at (-158.7, 153.9)
- added Y1: XTAL, Crystal:Crystal_SMD_3225-4Pin_3.2x2.5mm, B.Cu at (-153.7, 153.8)
Routing:
- net row0: track 0.00 -> 281.0 mm
- net row6: track 0.00 -> 279.9 mm
- net row2: track 0.00 -> 270.8 mm
- net row4: track 0.00 -> 266.0 mm
- net row7: track 0.00 -> 265.4 mm
- net row1: track 0.00 -> 262.0 mm
- net row3: track 0.00 -> 261.2 mm
- net row8: track 0.00 -> 251.7 mm
- net row5: track 0.00 -> 245.5 mm
- net row9: track 0.00 -> 210.5 mm
- net col7: track 0.00 -> 204.9 mm
- net col0: track 0.00 -> 197.2 mm
- net col5: track 0.00 -> 194.6 mm
- net col3: track 0.00 -> 178.2 mm
- net col1: track 0.00 -> 174.7 mm
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Other:
- copper layers 0 -> 2
