File: 66_ekip.kicad_sch (KiCad schematic)
At the start: 0 parts

Commit message: Matrix routed on the PCB
Parts:
- added C1, C2: 22p, Capacitor_SMD:C_0805_2012Metric, symbol Device:C_Small
- added C10, C11, C8, C9: 0.1u, Capacitor_SMD:C_0805_2012Metric, symbol Device:C_Small
- added C12, C13, C4, C6: 10u, Capacitor_SMD:C_0805_2012Metric, symbol Device:C_Small
- added C14: 100nF, Capacitor_SMD:C_0805_2012Metric, symbol Device:C_Small
- added C3, C5, C7: 1u, Capacitor_SMD:C_0805_2012Metric, symbol Device:C_Small
- added D70: D_Small, Diode_SMD:D_0805_2012Metric, symbol Device:D_Small
- added D71: LED, LED_SMD:LED_0805_2012Metric, symbol Device:LED
- added D72, D73, D74, D75, D76, D77: WS2812, LED_SMD:LED_WS2812_PLCC6_5.0x5.0mm_P1.6mm, symbol LED:WS2812
- added J1: BT LE, Connector_PinHeader_1.00mm:PinHeader_1x09_P1.00mm_Vertical, symbol Connector:Conn_01x09_Male
- added J2: AVR-ISP-6, Random_Keyb_Parts:Reset_Pretty, symbol Connector:AVR-ISP-6
- added J3: JST, Connector_JST:JST_SH_SM04B-SRSS-TB_1x04-1MP_P1.00mm_Horizontal, symbol Connector:Conn_01x04_Male
- added J4: BAT JST, Connector_JST:JST_PH_S2B-PH-SM4-TB_1x02-1MP_P2.00mm_Horizontal, symbol Connector:Conn_01x02_Male
- added R1, R2: 22, Resistor_SMD:R_0805_2012Metric, symbol Device:R_Small
- added R3: 100k, Resistor_SMD:R_0805_2012Metric, symbol Device:R_Small
- added R4, R6, R7: 10k, Resistor_SMD:R_0805_2012Metric, symbol Device:R_Small
- added R5: 1k, Resistor_SMD:R_0805_2012Metric, symbol Device:R_Small
- added R8: 480, Resistor_SMD:R_0805_2012Metric, symbol Device:R_Small
- added SW77: SW_Push, Button_Switch_SMD:SW_SPST_SKQG_WithStem, symbol Switch:SW_Push
- added U1: AP2112K-3.3, Package_TO_SOT_SMD:SOT-23-5, symbol Regulator_Linear:AP2112K-3.3
- added U2: ATmega32U4-AU, Package_QFP:TQFP-44_10x10mm_P0.8mm, symbol MCU_Microchip_ATmega:ATmega32U4-AU
- added U3: MCP73831-2-OT, Package_TO_SOT_SMD:SOT-23-5, symbol Battery_Management:MCP73831-2-OT
- added Y1: XTAL, Crystal:Crystal_SMD_3225-4Pin_3.2x2.5mm, symbol Device:Crystal_GND24_Small
Connections:
- new net: C3.1, U2.42 (AREF)
- new net: D74.1 (DOUT), D75.2 (DIN)
- new net: D73.1 (DOUT), D74.2 (DIN)
- new net: D72.2 (DIN), R8.1
- new net: R2.2, U2.3 (D-)
- new net: C7.1, U2.6 (UCAP)
- new net: D71.1 (K), R5.1
- new net: R5.2, U3.1 (STAT)
- new net: R4.1, U2.33 (~HWB~/PE2)
- new net: R7.1, U3.5 (PROG)
- new net: D76.1 (DOUT), D77.2 (DIN)
- new net: D75.1 (DOUT), D76.2 (DIN)
- new net: R1.2, U2.4 (D+)
- new net: R3.1, U1.3 (EN)
- new net: D72.1 (DOUT), D73.2 (DIN)
- new net +3V3: C10.1, C11.1, C12.1, C4.1, C5.1, C8.1, C9.1, U1.5 (VOUT), U2.14 (VCC), U2.2 (UVCC), U2.24 (AVCC), U2.34 (VCC), U2.44 (AVCC)
- new net +5V: C14.1, C6.1, D70.1 (K), D71.2 (A), D72.5 (VDD), D73.5 (VDD), D74.5 (VDD), D75.5 (VDD), D76.5 (VDD), D77.5 (VDD), J1.2 (Pin_2), J2.2 (VCC), J3.4 (Pin_4), R3.2, R6.1, U1.1 (VIN), U2.7 (VBUS), U3.4 (VDD)
- new net CS: J1.6 (Pin_6), U2.28 (PB4)
- new net D+: J3.2 (Pin_2), R1.1
- new net D-: J3.3 (Pin_3), R2.1
- new net DFU: J1.4 (Pin_4)
- new net GND: C1.2, C10.2, C11.2, C12.2, C13.2, C14.2, C2.2, C3.2, C4.2, C5.2, C6.2, C7.2, C8.2, C9.2, D72.6 (VSS), D73.6 (VSS), D74.6 (VSS), D75.6 (VSS), D76.6 (VSS), D77.6 (VSS), J1.1 (Pin_1), J2.6 (GND), J3.1 (Pin_1), J4.1 (Pin_1), R4.2, R7.2, SW77.1, U1.2 (GND), U2.15 (GND), U2.23 (GND), U2.35 (GND), U2.43 (GND), U2.5 (UGND), U3.2 (VSS), Y1.2, Y1.4
- new net IRQ: J1.5 (Pin_5), U2.1 (PE6)
- new net MISO: J1.8 (Pin_8), J2.1 (MISO), U2.11 (PB3)
- new net MOSI: J1.7 (Pin_7), J2.4 (MOSI), U2.10 (PB2)
- new net RGB_PIN: R8.2, U2.8 (PB0)
- new net RST: J1.3 (Pin_3), J2.5 (~RST), R6.2, SW77.2, U2.13 (~RESET)
- new net SCK: J1.9 (Pin_9), J2.3 (SCK), U2.9 (PB1)
- new net VBAT: C13.1, D70.2 (A), J4.2 (Pin_2), U3.3 (VBAT)
- new net XTAL1: C1.1, U2.17 (XTAL1), Y1.1
- new net XTAL2: C2.1, U2.16 (XTAL2), Y1.3
Other:
- added sheet matrix (matrix.kicad_sch)
